Commit message: Fix: fix the urdf file over
 - Edit the overall urdf
 - Create the new transmission file

File: src/agv_forklift_description/urdf/agv_forklift.gazebo.xacro (robot description, xacro)
@@ -1,16 +1,11 @@
 <?xml version="1.0"?>
 <robot xmlns:xacro="http://www.ros.org/wiki/xacro">
-  <xacro:property name="silver" value="Gazebo/Grey"/>
-  <xacro:property name="black" value="Gazebo/DarkGrey"/>
-  <xacro:property name="indigo" value="Gazebo/Indigo"/>
-  <xacro:property name="blue" value="Gazebo/Blue"/>
-  <xacro:property name="green" value="Gazebo/Green"/>
-  <xacro:property name="green_glow" value="Gazebo/GreenGlow"/>
-  <xacro:property name="yellow" value="Gazebo/Yellow"/>
-  <xacro:macro name="gazebo_common" params="link_name color mu_1 mu_2">
+  <xacro:macro name="gazebo_common" params="link_name color mu_1:=0 mu_2:=0 k_p:=0 k_d:=0">
     <gazebo reference="${link_name}_link">
       <material>${color}</material>
       <mu1>${mu_1}</mu1>
       <mu2>${mu_2}</mu2>
+      <kp>${k_p}</kp>
+      <kd>${k_d}</kd>
     </gazebo>
   </xacro:macro>

File: src/agv_forklift_description/urdf/agv_forklift.xacro (robot description, xacro)
@@ -2,7 +2,7 @@
 <robot name="agv_forklift" xmlns:xacro="http://www.ros.org/wiki/xacro">
   <xacro:include filename="$(find agv_forklift_description)/urdf/materials.xacro" />
-  <xacro:include filename="$(find agv_forklift_description)/urdf/agv_forklift.trans" />
   <xacro:include filename="$(find agv_forklift_description)/urdf/agv_forklift.gazebo.xacro" />
   <xacro:include filename="$(find agv_forklift_description)/urdf/wheels.urdf.xacro" />
+  <xacro:include filename="$(find agv_forklift_description)/urdf/agv_forklift.transmission.xacro" />
   <!-- The links -->
   <link name="base_link">
@@ -155,4 +155,15 @@
       </joint>
     </container>
+    <trans_container>
+      <transmission name="front_left_whole_rotate_joint_trans">
+        <type>transmission_interface/SimpleTransmission</type>
+        <actuator name="front_left_whole_rotate_joint_motor">
+          <mechanicalReduction>1</mechanicalReduction>
+        </actuator>
+        <joint name="front_left_whole_rotate_joint">
+          <hardwareInterface>hardware_interface/PositionJointInterface</hardwareInterface>
+        </joint>
+      </transmission>
+    </trans_container>
   </xacro:wheel_macro>
   <xacro:wheel_macro direction="front_right">
@@ -165,4 +176,15 @@
       </joint>
     </container>
+    <trans_container>
+      <transmission name="front_right_whole_rotate_joint_trans">
+        <type>transmission_interface/SimpleTransmission</type>
+        <actuator name="front_right_whole_rotate_joint_motor">
+          <mechanicalReduction>1</mechanicalReduction>
+        </actuator>
+        <joint name="front_right_whole_rotate_joint">
+          <hardwareInterface>hardware_interface/PositionJointInterface</hardwareInterface>
+        </joint>
+      </transmission>
+    </trans_container>
   </xacro:wheel_macro>
   <xacro:wheel_macro direction="back_left">
@@ -175,4 +197,15 @@
       </joint>
     </container>
+    <trans_container>
+      <transmission name="back_left_whole_rotate_joint_trans">
+        <type>transmission_interface/SimpleTransmission</type>
+        <actuator name="back_left_whole_rotate_joint_motor">
+          <mechanicalReduction>1</mechanicalReduction>
+        </actuator>
+        <joint name="back_left_whole_rotate_joint">
+          <hardwareInterface>hardware_interface/PositionJointInterface</hardwareInterface>
+        </joint>
+      </transmission>
+    </trans_container>
   </xacro:wheel_macro>
   <xacro:wheel_macro direction="back_right">
@@ -185,4 +218,15 @@
       </joint>
     </container>
+    <trans_container>
+      <transmission name="back_right_whole_rotate_joint_trans">
+        <type>transmission_interface/SimpleTransmission</type>
+        <actuator name="back_right_whole_rotate_joint_motor">
+          <mechanicalReduction>1</mechanicalReduction>
+        </actuator>
+        <joint name="back_right_whole_rotate_joint">
+          <hardwareInterface>hardware_interface/PositionJointInterface</hardwareInterface>
+        </joint>
+      </transmission>
+    </trans_container>
   </xacro:wheel_macro>
   <link name="top_lidar_link">
@@ -246,35 +290,34 @@
   </joint>
   <!-- The gazebo relevant -->
+  <gazebo>
+    <plugin name="gazebo_ros_control" filename="libgazebo_ros_control.so">
+      <robotNamespace>/</robotNamespace>
+    </plugin>
+  </gazebo>
   <xacro:gazebo_common link_name="base"
-                       color="${black}"
-                       mu_1="0"
-                       mu_2="0"/>
+                       color="${black}"/>
   <xacro:gazebo_common link_name="base_down_lidar_left"
-                       color="${indigo}"
-                       mu_1="0"
-                       mu_2="0"/>
+                       color="${indigo}"/>
   <xacro:gazebo_common link_name="base_down_lidar_right"
-                       color="${indigo}"
-                       mu_1="0"
-                       mu_2="0"/>
+                       color="${indigo}"/>
   <xacro:gazebo_common link_name="battery"
-                       color="${silver}"
-                       mu_1="0"
-                       mu_2="0"/>
+                       color="${silver}"/>
   <xacro:gazebo_common link_name="forklift_body"
-                       color="${blue}"
-                       mu_1="0"
-                       mu_2="0"/>
+                       color="${blue}"/>
   <xacro:gazebo_common link_name="beam"
-                       color="${silver}"
-                       mu_1="0"
-                       mu_2="0"/>
+                       color="${silver}"/>
   <xacro:gazebo_common link_name="fork"
                        color="${black}"
-                       mu_1="0.35"
-                       mu_2="0.35"/>
+                       mu_1="350.0"
+                       mu_2="320.0"
+                       k_p="10000000.0"
+                       k_d="0.0"/>
   <xacro:gazebo_common link_name="top_lidar"
                        color="${yellow}"
-                       mu_1="0.35"
-                       mu_2="0.35"/>
+                       mu_1="350.0"
+                       mu_2="320.0"
+                       k_p="10000000.0"
+                       k_d="0.0"/>
+  <!-- Transmissions -->
+  <xacro:forklift_transmission />
 </robot>

File: src/agv_forklift_description/urdf/materials.xacro (robot description, xacro)
@@ -1,6 +1,14 @@
 <?xml version="1.0" ?>
 <robot name="agv_forklift" xmlns:xacro="http://www.ros.org/wiki/xacro" >
-<material name="silver">
-  <color rgba="0.700 0.700 0.700 1.000"/>
-</material>
+  <!-- For gazebo -->>
+  <xacro:property name="silver" value="Gazebo/Grey"/>
+  <xacro:property name="black" value="Gazebo/DarkGrey"/>
+  <xacro:property name="indigo" value="Gazebo/Indigo"/>
+  <xacro:property name="blue" value="Gazebo/Blue"/>
+  <xacro:property name="green" value="Gazebo/Green"/>
+  <xacro:property name="green_glow" value="Gazebo/GreenGlow"/>
+  <xacro:property name="yellow" value="Gazebo/Yellow"/>
+  <material name="silver">
+    <color rgba="0.700 0.700 0.700 1.000"/>
+  </material>
 </robot>

File: src/agv_forklift_description/urdf/wheels.urdf.xacro (robot description, xacro)
@@ -2,5 +2,5 @@
 <robot xmlns:xacro="http://www.ros.org/wiki/xacro">
   <xacro:include filename="$(find agv_forklift_description)/urdf/agv_forklift.gazebo.xacro" />
-  <xacro:macro name="wheel_macro" params="direction **content">
+  <xacro:macro name="wheel_macro" params="direction **content **transmission">
     <!-- Links in the wheel -->
     <link name="${direction}_wheel_left_tyre_link">
@@ -147,29 +147,45 @@
     </joint>
     <xacro:insert_block name="content"/>
+    <xacro:insert_block name="transmission"/>
     <!-- Gazebo -->
     <xacro:gazebo_common link_name="${direction}_wheel_left_tyre"
                          color="${black}"
-                         mu_1="0.8"
-                         mu_2="0.8"/>
+                         mu_1="800.0"
+                         mu_2="800.0"
+                         k_p="10000000.0"
+                         k_d="0.0"/>
     <xacro:gazebo_common link_name="${direction}_wheel_right_tyre"
                          color="${black}"
-                         mu_1="0.8"
-                         mu_2="0.8"/>
+                         mu_1="800.0"
+                         mu_2="800.0"
+                         k_p="10000000.0"
+                         k_d="0.0"/>
     <xacro:gazebo_common link_name="${direction}_wheel_left_side"
-                         color="${silver}"
-                         mu_1="0"
-                         mu_2="0"/>
+                         color="${silver}"/>
     <xacro:gazebo_common link_name="${direction}_wheel_right_side"
-                         color="${silver}"
-                         mu_1="0"
-                         mu_2="0"/>
+                         color="${silver}"/>
     <xacro:gazebo_common link_name="${direction}_wheel_body"
-                         color="${green}"
-                         mu_1="0"
-                         mu_2="0"/>
+                         color="${green}"/>
     <xacro:gazebo_common link_name="{direction}_wheel_body_wheel_lid"
-                         color="${green}"
-                         mu_1="0"
-                         mu_2="0"/>
+                         color="${green}"/>
+    <!-- Transmissions -->
+    <transmission name="${direction}_left_rotate_joint_trans">
+      <type>transmission_interface/SimpleTransmission</type>
+      <actuator name="${direction}_left_rotate_joint_motor">
+          <mechanicalReduction>1</mechanicalReduction>
+      </actuator>
+      <joint name="${direction}_left_rotate_joint">
+          <hardwareInterface>VelocityJointInterface</hardwareInterface>
+      </joint>
+    </transmission>
+    <transmission name="${direction}_right_rotate_joint_trans">
+      <type>transmission_interface/SimpleTransmission</type>
+      <actuator name="${direction}_right_rotate_joint_motor">
+          <mechanicalReduction>1</mechanicalReduction>
+      </actuator>
+      <joint name="${direction}_right_rotate_joint">
+          <hardwareInterface>VelocityJointInterface</hardwareInterface>
+      </joint>
+    </transmission>
   </xacro:macro>
 </robot>
