Commit message: Finish the move part. One bug: param can not load

File: src/agv_forklift_description/urdf/wheels.urdf.xacro (robot description, xacro)
@@ -128,5 +128,5 @@
       <parent link="${direction}_wheel_body_link"/>
       <child link="${direction}_wheel_left_side_link"/>
-      <axis xyz="-0.0 1.0 0.0"/>
+      <axis xyz="0.0 1.0 0.0"/>
     </joint>
     <joint name="${direction}_right_tyre_joint" type="fixed">
@@ -139,5 +139,5 @@
       <parent link="${direction}_wheel_body_link"/>
       <child link="${direction}_wheel_right_side_link"/>
-      <axis xyz="-0.0 1.0 0.0"/>
+      <axis xyz="0.0 1.0 0.0"/>
     </joint>
     <joint name="${direction}_wheel_lid_joint" type="fixed">
