Commit message: Lift move part finish. But the car will fly when collide

File: src/agv_forklift_description/urdf/agv_forklift.xacro (robot description, xacro)
@@ -1,8 +1,8 @@
 <?xml version="1.0" ?>
-<robot name="agv_forklift" xmlns:xacro="http://www.ros.org/wiki/xacro">
-  <xacro:include filename="$(find agv_forklift_description)/urdf/materials.xacro" />
-  <xacro:include filename="$(find agv_forklift_description)/urdf/agv_forklift.gazebo.xacro" />
-  <xacro:include filename="$(find agv_forklift_description)/urdf/wheels.urdf.xacro" />
-  <xacro:include filename="$(find agv_forklift_description)/urdf/agv_forklift.transmission.xacro" />
+<robot xmlns:xacro="http://www.ros.org/wiki/xacro" name="agv_forklift">
+  <xacro:include filename="$(find agv_forklift_description)/urdf/materials.xacro"/>
+  <xacro:include filename="$(find agv_forklift_description)/urdf/agv_forklift.gazebo.xacro"/>
+  <xacro:include filename="$(find agv_forklift_description)/urdf/wheels.urdf.xacro"/>
+  <xacro:include filename="$(find agv_forklift_description)/urdf/agv_forklift.transmission.xacro"/>
   <!-- The links -->
   <link name="base_link">
@@ -282,5 +282,5 @@
     <axis xyz="0.0 0.0 1.0"/>
     <!-- TODO: effort fill -->
-    <limit upper="1.4" lower="0.0" effort="100" velocity="0.1"/>
+    <limit upper="1.6" lower="0.0" effort="1000" velocity="1"/>
   </joint>
   <joint name="body_lidar_joint" type="fixed">
@@ -297,41 +297,43 @@
   <xacro:gazebo_common link_name="base"
                        color="${black}"
-                       mu_1="300"
-                       mu_2="300"
-                       k_p="10000000.0"
-                       k_d="100.0"/>
+                       mu_1="0.35"
+                       mu_2="0.35"
+                       k_p="100.0"
+                       k_d="1.0"/>
   <xacro:gazebo_common link_name="base_down_lidar_left"
                        color="${indigo}"
-                       k_p="10000000.0"
-                       k_d="100.0"/>
+                       k_p="100.0"
+                       k_d="1.0"/>
   <xacro:gazebo_common link_name="base_down_lidar_right"
                        color="${indigo}"
-                       k_p="10000000.0"
-                       k_d="100.0"/>
+                       k_p="100.0"
+                       k_d="1.0"/>
   <xacro:gazebo_common link_name="battery"
                        color="${silver}"
-                       k_p="10000000.0"
-                       k_d="100.0"/>
+                       k_p="100.0"
+                       k_d="1.0"/>
   <xacro:gazebo_common link_name="forklift_body"
                        color="${blue}"
-                       k_p="10000000.0"
-                       k_d="100.0"/>
+                       k_p="100.0"
+                       k_d="1.0"/>
   <xacro:gazebo_common link_name="beam"
                        color="${silver}"
+                       mu_1="0.35"
+                       mu_2="0.35"
                        k_p="10000000.0"
                        k_d="100.0"/>
   <xacro:gazebo_common link_name="fork"
                        color="${black}"
-                       mu_1="350.0"
-                       mu_2="320.0"
-                       k_p="10000000.0"
-                       k_d="0.0"/>
+                       mu_1="0.35"
+                       mu_2="0.35"
+                       k_p="100.0"
+                       k_d="1.0"/>
   <xacro:gazebo_common link_name="top_lidar"
                        color="${yellow}"
-                       mu_1="350.0"
-                       mu_2="320.0"
-                       k_p="10000000.0"
-                       k_d="0.0"/>
+                       mu_1="0.35"
+                       mu_2="0.35"
+                       k_p="100.0"
+                       k_d="1.0"/>
   <!-- Transmissions -->
-  <xacro:forklift_transmission />
+  <xacro:forklift_transmission/>
 </robot>

Commit message: New begin

File: src/agv_forklift_description/urdf/agv_forklift.xacro (robot description, xacro)
@@ -6,5 +6,6 @@
   <xacro:include filename="$(find agv_forklift_description)/urdf/agv_forklift.transmission.xacro"/>
   <!-- The links -->
-  <link name="base_link">
+  <link name="base_link"/>
+  <link name="chassis_link">
     <inertial>
       <origin xyz="-1.113481469298291 0.0 0.05983225879940115" rpy="0 0 0"/>
@@ -129,5 +130,5 @@
     <inertial>
       <origin xyz="-0.6484229539416837 0.4723008933333786 -1.6470003187088946" rpy="0 0 0"/>
-      <mass value="365.22311207175414"/>
+      <mass value="36.22311207175414"/>
       <inertia ixx="63.839107" iyy="87.82671" izz="138.209861" ixy="-0.000165" iyz="-8.9e-05" ixz="-14.023649"/>
     </inertial>
@@ -150,5 +151,5 @@
       <joint name="front_left_whole_rotate_joint" type="continuous">
         <origin xyz="-0.416667 0.4 0.1" rpy="0 0 0"/>
-        <parent link="base_link"/>
+        <parent link="chassis_link"/>
         <child link="front_left_wheel_body_link"/>
         <axis xyz="0.0 0.0 -1.0"/>
@@ -171,5 +172,5 @@
       <joint name="front_right_whole_rotate_joint" type="continuous">
         <origin xyz="-0.416667 -0.4 0.1" rpy="0 0 0"/>
-        <parent link="base_link"/>
+        <parent link="chassis_link"/>
         <child link="front_right_wheel_body_link"/>
         <axis xyz="0.0 0.0 -1.0"/>
@@ -192,5 +193,5 @@
       <joint name="back_left_whole_rotate_joint" type="continuous">
         <origin xyz="-2.0833337 0.4 0.1" rpy="0 0 0"/>
-        <parent link="base_link"/>
+        <parent link="chassis_link"/>
         <child link="back_left_wheel_body_link"/>
         <axis xyz="0.0 0.0 -1.0"/>
@@ -213,5 +214,5 @@
       <joint name="back_right_whole_rotate_joint" type="continuous">
         <origin xyz="-2.0833337 -0.4 0.1" rpy="0 0 0"/>
-        <parent link="base_link"/>
+        <parent link="chassis_link"/>
         <child link="back_right_wheel_body_link"/>
         <axis xyz="0.0 0.0 -1.0"/>
@@ -251,22 +252,27 @@
   </link>
   <!-- The joints -->
+  <joint name="base_chassis_joint" type="fixed">
+    <origin xyz="0 0 0" rpy="0 0 0"/>
+    <parent link="base_link"/>
+    <child link="chassis_link"/>
+  </joint>
   <joint name="base_down_lidar_right_joint" type="fixed">
     <origin xyz="-0.055934 -0.456066 0.055" rpy="0 0 0"/>
-    <parent link="base_link"/>
+    <parent link="chassis_link"/>
     <child link="down_lidar_link_right"/>
   </joint>
   <joint name="base_down_lidar_left_joint" type="fixed">
     <origin xyz="-0.055934 0.456066 0.055" rpy="0 0 0"/>
-    <parent link="base_link"/>
+    <parent link="chassis_link"/>
     <child link="down_lidar_link_left"/>
   </joint>
   <joint name="base_battery_joint" type="fixed">
     <origin xyz="-0.05 0.0 0.105" rpy="0 0 0"/>
-    <parent link="base_link"/>
+    <parent link="chassis_link"/>
     <child link="battery_link"/>
   </joint>
   <joint name="base_body_joint" type="fixed">
     <origin xyz="0.0 0.0 0.105" rpy="0 0 0"/>
-    <parent link="base_link"/>
+    <parent link="chassis_link"/>
     <child link="forklift_body_link"/>
   </joint>
@@ -277,6 +283,6 @@
   </joint>
   <joint name="beam_fork_slide_joint" type="prismatic">
-    <origin xyz="0.075 -0.9823 0.56" rpy="0 0 0"/>
-    <parent link="beam_link"/>
+    <origin xyz="-0.575 -0.4732 1.895" rpy="0 0 0"/>
+    <parent link="base_link"/>
     <child link="fork_link"/>
     <axis xyz="0.0 0.0 1.0"/>
@@ -295,44 +301,44 @@
     </plugin>
   </gazebo>
-  <xacro:gazebo_common link_name="base"
+  <xacro:gazebo_common link_name="chassis"
                        color="${black}"
                        mu_1="0.35"
                        mu_2="0.35"
-                       k_p="100.0"
-                       k_d="1.0"/>
+                       k_p="0.0"
+                       k_d="0.0"/>
   <xacro:gazebo_common link_name="base_down_lidar_left"
                        color="${indigo}"
-                       k_p="100.0"
-                       k_d="1.0"/>
+                       k_p="0.0"
+                       k_d="0.0"/>
   <xacro:gazebo_common link_name="base_down_lidar_right"
                        color="${indigo}"
-                       k_p="100.0"
-                       k_d="1.0"/>
+                       k_p="0.0"
+                       k_d="0.0"/>
   <xacro:gazebo_common link_name="battery"
                        color="${silver}"
-                       k_p="100.0"
-                       k_d="1.0"/>
+                       k_p="0.0"
+                       k_d="0.0"/>
   <xacro:gazebo_common link_name="forklift_body"
                        color="${blue}"
-                       k_p="100.0"
-                       k_d="1.0"/>
+                       k_p="0.0"
+                       k_d="0.0"/>
   <xacro:gazebo_common link_name="beam"
                        color="${silver}"
                        mu_1="0.35"
                        mu_2="0.35"
-                       k_p="10000000.0"
-                       k_d="100.0"/>
+                       k_p="0.0"
+                       k_d="0.0"/>
   <xacro:gazebo_common link_name="fork"
                        color="${black}"
                        mu_1="0.35"
                        mu_2="0.35"
-                       k_p="100.0"
-                       k_d="1.0"/>
+                       k_p="0.0"
+                       k_d="0.0"/>
   <xacro:gazebo_common link_name="top_lidar"
                        color="${yellow}"
                        mu_1="0.35"
                        mu_2="0.35"
-                       k_p="100.0"
-                       k_d="1.0"/>
+                       k_p="0.0"
+                       k_d="0.0"/>
   <!-- Transmissions -->
   <xacro:forklift_transmission/>

File: src/agv_forklift_description/urdf/wheels.urdf.xacro (robot description, xacro)
@@ -181,8 +181,8 @@
       <type>transmission_interface/SimpleTransmission</type>
       <actuator name="${direction}_left_rotate_joint_motor">
-          <mechanicalReduction>1</mechanicalReduction>
+        <mechanicalReduction>1</mechanicalReduction>
       </actuator>
       <joint name="${direction}_left_rotate_joint">
-          <hardwareInterface>hardware_interface/EffortJointInterface</hardwareInterface>
+        <hardwareInterface>hardware_interface/EffortJointInterface</hardwareInterface>
       </joint>
     </transmission>
@@ -190,8 +190,8 @@
       <type>transmission_interface/SimpleTransmission</type>
       <actuator name="${direction}_right_rotate_joint_motor">
-          <mechanicalReduction>1</mechanicalReduction>
+        <mechanicalReduction>1</mechanicalReduction>
       </actuator>
       <joint name="${direction}_right_rotate_joint">
-          <hardwareInterface>hardware_interface/EffortJointInterface</hardwareInterface>
+        <hardwareInterface>hardware_interface/EffortJointInterface</hardwareInterface>
       </joint>
     </transmission>

Commit message: Finish Navigation

File: src/agv_forklift_description/urdf/agv_forklift.xacro (robot description, xacro)
@@ -254,5 +254,5 @@
   <!-- The joints -->
   <joint name="base_chassis_joint" type="fixed">
-    <origin xyz="0 0 0" rpy="0 0 0"/>
+    <origin xyz="1.25 0 0" rpy="0 0 0"/>
     <parent link="base_link"/>
     <child link="chassis_link"/>
@@ -284,5 +284,5 @@
   </joint>
   <joint name="beam_fork_slide_joint" type="prismatic">
-    <origin xyz="-0.575 -0.4732 1.895" rpy="0 0 0"/>
+    <origin xyz="0.675 -0.4732 1.895" rpy="0 0 0"/>
     <parent link="base_link"/>
     <child link="fork_link"/>
@@ -292,5 +292,5 @@
   </joint>
   <joint name="body_lidar_joint" type="fixed">
-    <origin xyz="-0.35 -0.0 1.835" rpy="0 0 0"/>
+    <origin xyz="-0.35 -0.0 1.845" rpy="0 0 0"/>
     <parent link="forklift_body_link"/>
     <child link="top_lidar_link"/>
